File: fsoc-tx/tx_mcu_clock.kicad_sch (KiCad schematic)
At the start: 31 parts, among them J3 FTSH-105-01-L-DV-K, SW1 SW_RESET, SW2 USB_BOOT, U3 RP2354A, Y1 ABM8-272-T3, Y3 SiT5346

Commit message: manufacturer part number for Sit5346
Parts:
- Y3: JLCPCB Part (none) -> TBD - Global Sourcing if not stocked; MPN (none) -> TBD - SiT5346 10MHz 3.3V LVCMOS DCTCXO
Changed lines of the file:
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@@
 			)
 		)
-		(property "Description" "10-pin 5.0x3.2 mm precision DCTCXO, I2C-controlled, LVCMOS clock output"
+		(property "Description" "SiT5346 DCTCXO, 10.000000 MHz, 3.3 V, LVCMOS, ±0.1 ppm, industrial, I2C-controlled"
 			(at 223.52 110.49 0)
 			(hide yes)
@@
 			(at 223.52 110.49 0)
 			(hide yes)
+			(show_name no)
+			(do_not_autoplace no)
+			(effects
+				(font
+					(size 1.27 1.27)
+				)
+			)
+		)
+		(property "MPN" "TBD - SiT5346 10MHz 3.3V LVCMOS DCTCXO"
+			(at 223.52 110.49 0)
+			(hide yes)
+			(show_name no)
+			(do_not_autoplace no)
+			(effects
+				(font
+					(size 1.27 1.27)
+				)
+			)
+		)
+		(property "JLCPCB Part" "TBD - Global Sourcing if not stocked"
+			(at 223.52 110.49 0)
+			(hide yes)
