File: fsoc-tx/tx_power_usb.kicad_sch (KiCad schematic)
At the start: 9 parts, among them J1 USB4105-GF-A, J2 B8B-PH-K-S, U1 USBLC6-2SC6, U2 AP2112K-3.3

Commit message: TX ROOT: laser + host IO
Changed lines of the file:
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@@
+		)
+	)
+	(label "SYS_5V"
+		(at 189.23 67.31 180)
+		(effects
+			(font
+				(size 1.27 1.27)
+			)
+			(justify right bottom)
 		)
 	)
 	(hierarchical_label "USB_DP"
-		(shape input)
+		(shape bidirectional)
 		(at 133.35 82.55 0)
 		(effects
@@
 	)
 	(hierarchical_label "USB_DM"
-		(shape input)
+		(shape bidirectional)
 		(at 133.35 80.01 0)
 		(effects
@@
 	)
 	(hierarchical_label "PPS_OUT"
-		(shape output)
+		(shape input)
 		(at 162.56 119.38 270)
 		(effects
@@
 	)
 	(hierarchical_label "HOST_READY"
-		(shape input)
+		(shape output)
 		(at 167.64 119.38 270)
 		(effects
@@
 		)
 	)
-	(hierarchical_label "SYS_5V"
+	(hierarchical_label "HOST_UART_RX"
 		(shape output)
-		(at 189.23 67.31 180)
-		(effects
-			(font
-				(size 1.27 1.27)
-			)
-			(justify right)
-		)
-	)
-	(hierarchical_label "HOST_UART_RX"
-		(shape input)
 		(at 147.32 119.38 270)
 		(effects
@@
 	)
 	(hierarchical_label "HOST_UART_TX"
-		(shape output)
+		(shape input)
 		(at 142.24 119.38 270)
 		(effects

Commit message: TX: fixing unassigned footprints
Parts:
- C1, C2: footprint (none) -> Capacitor_SMD:C_0805_2012Metric
- R1, R2: footprint (none) -> Resistor_SMD:R_0603_1608Metric
Changed lines of the file:
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@@
 			)
 		)
-		(property "Footprint" ""
+		(property "Footprint" "Resistor_SMD:R_0603_1608Metric"
 			(at 101.6 74.168 90)
 			(hide yes)
@@
 			)
 		)
-		(property "Footprint" ""
+		(property "Footprint" "Capacitor_SMD:C_0805_2012Metric"
 			(at 197.8152 77.47 0)
 			(hide yes)
@@
 			)
 		)
-		(property "Footprint" ""
+		(property "Footprint" "Resistor_SMD:R_0603_1608Metric"
 			(at 101.6 76.708 90)
 			(hide yes)
@@
 			)
 		)
-		(property "Footprint" ""
+		(property "Footprint" "Capacitor_SMD:C_0805_2012Metric"
 			(at 223.2152 77.47 0)
 			(hide yes)

Commit message: TX PCB: DONE
Parts:
- J1: footprint Connector_USB:USB_C_Receptacle_GCT_USB4105-xx-A_16P_TopMnt_Horizontal -> fsoc_footprints:TYPE-C-31-M-14
Connections:
- net USB_CONN_DP: now reaches J1.A6 (D+), J1.B6 (D+), U1.3 (I/O2)
- net USB_CONN_DN: now reaches J1.A7 (D-), J1.B7 (D-), U1.1 (I/O1)
- net USB_DM renamed USB_DN
Changed lines of the file:
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@@
+	(wire
+		(pts
+			(xy 101.6 82.55) (xy 101.6 80.01)
+		)
+		(stroke
+			(width 0)
+			(type default)
+		)
+	)
 	(wire
 		(pts
@@
 		(pts
 			(xy 133.35 62.23) (xy 133.35 67.31)
-		)
-		(stroke
-			(width 0)
-			(type default)
-		)
-	)
-	(wire
-		(pts
-			(xy 101.6 80.01) (xy 101.6 82.55)
 		)
 		(stroke
@@
 		)
 	)
+	(label "USB_CONN_DP"
+		(at 104.14 85.09 0)
+		(effects
+			(font
+				(size 1.27 1.27)
+			)
+			(justify left bottom)
+		)
+	)
 	(label "VIN_HOST_5V"
 		(at 165.1 85.09 0)
@@
 			)
 			(justify right bottom)
+		)
+	)
+	(label "USB_CONN_DN"
+		(at 101.6 82.55 0)
+		(effects
+			(font
+				(size 1.27 1.27)
+			)
+			(justify left bottom)
 		)
 	)
@@
 		)
 	)
-	(hierarchical_label "USB_DM"
+	(hierarchical_label "USB_DN"
 		(shape bidirectional)
 		(at 133.35 80.01 0)
@@
 			)
 		)
-		(property "Footprint" "Connector_USB:USB_C_Receptacle_GCT_USB4105-xx-A_16P_TopMnt_Horizontal"
+		(property "Footprint" "fsoc_footprints:TYPE-C-31-M-14"
 			(at 86.36 82.55 0)
 			(hide yes)

Commit message: manufacturing files
Parts:
- J2: footprint Connector_JST:JST_PH_B8B-PH-K_1x08_P2.00mm_Vertical -> Connector_PinHeader_2.54mm:PinHeader_1x08_P2.54mm_Vertical
Changed lines of the file:
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@@
 			)
 		)
-		(property "Footprint" "Connector_JST:JST_PH_B8B-PH-K_1x08_P2.00mm_Vertical"
+		(property "Footprint" "Connector_PinHeader_2.54mm:PinHeader_1x08_P2.54mm_Vertical"
 			(at 175.26 96.52 0)
 			(hide yes)
