File: fsoc-rx/rx_monitor.kicad_sch (KiCad schematic)
At the start: 0 parts

Commit message: RX ROOT: optical AFE
Parts:
- added C27: 10 nF, symbol Device:C
- added R14: 10 kΩ, symbol Device:R
Connections:
- new net GND: C27.2
- new net RX_LEVEL_MON: C27.1, R14.2
- new net TIA_OUT: R14.1

Commit message: RX: footprint assignments
Parts:
- C27: footprint (none) -> Capacitor_SMD:C_0603_1608Metric
- R14: footprint (none) -> Resistor_SMD:R_0603_1608Metric
Changed lines of the file:
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@@
 			)
 		)
-		(property "Footprint" ""
+		(property "Footprint" "Capacitor_SMD:C_0603_1608Metric"
 			(at 147.0152 102.87 0)
 			(hide yes)
@@
 			)
 		)
-		(property "Footprint" ""
+		(property "Footprint" "Resistor_SMD:R_0603_1608Metric"
 			(at 134.62 91.948 90)
 			(hide yes)
