File: fsoc-rx/rx_optical_afe.kicad_sch (KiCad schematic)
At the start: 13 parts, among them U5 OPA320AIDBVR, U6 TLV3201AIDBVR

Commit message: RX ROOT: optical AFE
Parts:
- renumbered C25 to C23, C23 to C24, C26 to C25, C24 to C26, Cf to Cf1, R13 to R12, R12 to R13, Rf to Rf1
Changed lines of the file:
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@@
 		(in_pos_files yes)
 		(dnp no)
-		(property "Reference" "#PWR034"
+		(property "Reference" "#PWR045"
 			(at 203.2 99.06 0)
 			(hide yes)
@@
 			(project "fsoc-rx"
 				(path "/84f983f4-ce6f-4382-bffe-129758307136/dc9b08a1-9ab8-4ff8-8f0e-d76c02b41618"
-					(reference "#PWR034")
+					(reference "#PWR045")
 					(unit 1)
 				)
@@
 		(dnp no)
 		(fields_autoplaced yes)
-		(property "Reference" "#PWR039"
+		(property "Reference" "#PWR041"
 			(at 135.89 130.81 0)
 			(hide yes)
@@
 			(project "fsoc-rx"
 				(path "/84f983f4-ce6f-4382-bffe-129758307136/dc9b08a1-9ab8-4ff8-8f0e-d76c02b41618"
-					(reference "#PWR039")
+					(reference "#PWR041")
 					(unit 1)
 				)
@@
 		(in_pos_files yes)
 		(dnp no)
-		(property "Reference" "C24"
+		(property "Reference" "C26"
 			(at 193.04 86.614 90)
 			(show_name no)
@@
 			(project "fsoc-rx"
 				(path "/84f983f4-ce6f-4382-bffe-129758307136/dc9b08a1-9ab8-4ff8-8f0e-d76c02b41618"
-					(reference "C24")
+					(reference "C26")
 					(unit 1)
 				)
@@
 		(dnp no)
 		(fields_autoplaced yes)
-		(property "Reference" "#PWR038"
+		(property "Reference" "#PWR039"
 			(at 118.11 130.81 0)
 			(hide yes)
@@
 			(project "fsoc-rx"
 				(path "/84f983f4-ce6f-4382-bffe-129758307136/dc9b08a1-9ab8-4ff8-8f0e-d76c02b41618"
-					(reference "#PWR038")
+					(reference "#PWR039")
 					(unit 1)
 				)
@@
 		(in_pos_files yes)
 		(dnp no)
-		(property "Reference" "Rf"
+		(property "Reference" "Rf1"
 			(at 156.21 107.95 90)
 			(show_name no)
@@
 			(project "fsoc-rx"
 				(path "/84f983f4-ce6f-4382-bffe-129758307136/dc9b08a1-9ab8-4ff8-8f0e-d76c02b41618"
-					(reference "Rf")
+					(reference "Rf1")
 					(unit 1)
 				)
@@
 		(dnp no)
 		(fields_autoplaced yes)
-		(property "Reference" "#PWR037"
+		(property "Reference" "#PWR042"
 			(at 143.51 113.03 0)
 			(hide yes)
@@
 			(project "fsoc-rx"
 				(path "/84f983f4-ce6f-4382-bffe-129758307136/dc9b08a1-9ab8-4ff8-8f0e-d76c02b41618"
-					(reference "#PWR037")
+					(reference "#PWR042")
 					(unit 1)
 				)
@@
 		(dnp no)
 		(fields_autoplaced yes)
-		(property "Reference" "#PWR040"
+		(property "Reference" "#PWR038"
 			(at 104.14 107.95 0)
 			(hide yes)
@@
 			(project "fsoc-rx"
 				(path "/84f983f4-ce6f-4382-bffe-129758307136/dc9b08a1-9ab8-4ff8-8f0e-d76c02b41618"
-					(reference "#PWR040")
+					(reference "#PWR038")
 					(unit 1)
 				)
@@
 		(dnp no)
 		(fields_autoplaced yes)
-		(property "Reference" "R13"
+		(property "Reference" "R12"
 			(at 168.91 76.2 90)
 			(show_name no)
@@
 			(project "fsoc-rx"
 				(path "/84f983f4-ce6f-4382-bffe-129758307136/dc9b08a1-9ab8-4ff8-8f0e-d76c02b41618"
-					(reference "R13")
+					(reference "R12")
 					(unit 1)
 				)
@@
 		(dnp no)
 		(fields_autoplaced yes)
-		(property "Reference" "R12"
+		(property "Reference" "R13"
 			(at 166.37 87.63 90)
 			(show_name no)
@@
 			(project "fsoc-rx"
 				(path "/84f983f4-ce6f-4382-bffe-129758307136/dc9b08a1-9ab8-4ff8-8f0e-d76c02b41618"
-					(reference "R12")
+					(reference "R13")
 					(unit 1)
 				)
@@
 		(dnp no)
 		(fields_autoplaced yes)
-		(property "Reference" "#PWR042"
+		(property "Reference" "#PWR046"
 			(at 207.01 90.17 0)
 			(hide yes)
@@
 			(project "fsoc-rx"
 				(path "/84f983f4-ce6f-4382-bffe-129758307136/dc9b08a1-9ab8-4ff8-8f0e-d76c02b41618"
-					(reference "#PWR042")
+					(reference "#PWR046")
 					(unit 1)
 				)
@@
 		(in_pos_files yes)
 		(dnp no)
-		(property "Reference" "Cf"
+		(property "Reference" "Cf1"
 			(at 156.21 112.014 90)
 			(show_name no)
@@
 			(project "fsoc-rx"
 				(path "/84f983f4-ce6f-4382-bffe-129758307136/dc9b08a1-9ab8-4ff8-8f0e-d76c02b41618"
-					(reference "Cf")
+					(reference "Cf1")
 					(unit 1)
 				)
@@
 		(dnp no)
 		(fields_autoplaced yes)
-		(property "Reference" "#PWR041"
+		(property "Reference" "#PWR043"
 			(at 172.72 99.06 0)
 			(hide yes)
@@
 			(project "fsoc-rx"
 				(path "/84f983f4-ce6f-4382-bffe-129758307136/dc9b08a1-9ab8-4ff8-8f0e-d76c02b41618"
-					(reference "#PWR041")
+					(reference "#PWR043")
 					(unit 1)
 				)
@@
 		(dnp no)
 		(fields_autoplaced yes)
-		(property "Reference" "C25"
+		(property "Reference" "C23"
 			(at 139.7 116.8399 0)
 			(show_name no)
@@
 			(project "fsoc-rx"
 				(path "/84f983f4-ce6f-4382-bffe-129758307136/dc9b08a1-9ab8-4ff8-8f0e-d76c02b41618"
-					(reference "C25")
+					(reference "C23")
 					(unit 1)
 				)
@@
 		(in_pos_files yes)
 		(dnp no)
-		(property "Reference" "C26"
+		(property "Reference" "C25"
 			(at 184.15 78.994 90)
 			(show_name no)
@@
 			(project "fsoc-rx"
 				(path "/84f983f4-ce6f-4382-bffe-129758307136/dc9b08a1-9ab8-4ff8-8f0e-d76c02b41618"
-					(reference "C26")
+					(reference "C25")
 					(unit 1)
 				)
@@
 		(dnp no)
 		(fields_autoplaced yes)
-		(property "Reference" "#PWR036"
+		(property "Reference" "#PWR040"
 			(at 127 99.06 0)
 			(hide yes)
@@
 			(project "fsoc-rx"
 				(path "/84f983f4-ce6f-4382-bffe-129758307136/dc9b08a1-9ab8-4ff8-8f0e-d76c02b41618"
-					(reference "#PWR036")
+					(reference "#PWR040")
 					(unit 1)
 				)
@@
 		(dnp no)
 		(fields_autoplaced yes)
-		(property "Reference" "C23"
+		(property "Reference" "C24"
 			(at 137.16 85.09 90)
 			(show_name no)
@@
 			(project "fsoc-rx"
 				(path "/84f983f4-ce6f-4382-bffe-129758307136/dc9b08a1-9ab8-4ff8-8f0e-d76c02b41618"
-					(reference "C23")
+					(reference "C24")
 					(unit 1)
 				)
@@
 		(dnp no)
 		(fields_autoplaced yes)
-		(property "Reference" "#PWR035"
+		(property "Reference" "#PWR044"
 			(at 189.23 111.76 0)
 			(hide yes)
@@
 			(project "fsoc-rx"
 				(path "/84f983f4-ce6f-4382-bffe-129758307136/dc9b08a1-9ab8-4ff8-8f0e-d76c02b41618"
-					(reference "#PWR035")
-					(unit 1)
-				)
+					(reference "#PWR044")
+					(unit 1)
+				)

Commit message: RX: footprint assignments
Parts:
- C23: footprint (none) -> Capacitor_SMD:C_0805_2012Metric
- C24, C25, C26: footprint (none) -> Capacitor_SMD:C_0603_1608Metric
- C28: renamed from Cf1; footprint (none) -> Capacitor_SMD:C_0603_1608Metric
- R10, R11, R12, R13: footprint (none) -> Resistor_SMD:R_0603_1608Metric
- R15: renamed from Rf1; footprint (none) -> Resistor_SMD:R_0603_1608Metric
Other:
- moved on the sheet: C23, C24, C25, C26, C28, D1, R10, R11, R12, R13, R15

Commit message: Manufacturing files
Parts:
- D1: MPN (none) -> BPW34; MPN: BPW34 -> (none); Manufacturer (none) -> Vishay Semiconductors; Manufacturer: Vishay Semiconductors -> (none)
