File: fsoc-rx/fsoc-rx.kicad_pcb (KiCad board)
At the start: 4 copper layers, 49.6 x 40 mm, 60 parts, among them J1 USB4105-GF-A, J2 B8B-PH-K-S, J3 FTSH-105-01-L-DV-K, J4 Conn_01x03, SW1 SW_RESET, SW2 USB_BOOT, U1 USBLC6-2SC6, U2 AP2112K-3.3, U3 TPS7A2033PDBVR, U4 RP2354A, U5 OPA320AIDBVR, U6 TLV3201AIDBVR, Y1 ABM8-272-T3, Y2 ASTX-H11-10.000MHz-T

Commit message: RX PCB: SiT5346
Parts:
- added C29: 100 nF, Capacitor_SMD:C_0603_1608Metric, F.Cu at (151.0, 95.5)
- added J5: Conn_01x02, Connector_PinHeader_2.54mm:PinHeader_1x02_P2.54mm_Vertical, F.Cu at (148.3, 101.0)
- C19: value 10 nF -> 10 µF; footprint Capacitor_SMD:C_0603_1608Metric -> Capacitor_SMD:C_0805_2012Metric
- Y2: value ASTX-H11-10.000MHz-T -> SiT5346; footprint fsoc_footprints:ASTX-H11_3225 -> fsoc_footprints:SiT5346_5.0x3.2mm_10L
- moved C19 27.7 mm to (154.3, 97.0), turned to -90 degrees
- moved Y2 25.5 mm to (148.0, 95.5), turned to 0 degrees
- moved C16 20.7 mm to (157.0, 114.0)
- moved C1 15.4 mm to (140.5, 91.5)
- moved C10 15.4 mm to (144.5, 87.0)
- moved C11 15.4 mm to (172.5, 101.5)
- moved C12 15.4 mm to (172.5, 99.5)
- moved C13 15.4 mm to (171.0, 108.0)
- moved C14 15.4 mm to (135.5, 89.5)
- moved C15 15.4 mm to (151.5, 86.0)
- moved C17 15.4 mm to (159.0, 84.0)
- moved C18 15.4 mm to (150.0, 86.0)
- moved C2 15.4 mm to (129.0, 83.5)
- moved C20 15.4 mm to (171.0, 106.5)
- moved C21 15.4 mm to (161.0, 84.0)
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Connections:
- U4 pad 16: /RX_MCU_CLOCK/TCXO_10M -> /RX_MCU_CLOCK/REF_10M
- Y2 pad 1: /+3V3_DIG -> unconnected-(Y2-OE/NC-Pad1)
- Y2 pad 2: GND -> /HOST_I2C_SCL
- Y2 pad 3: /RX_MCU_CLOCK/TCXO_10M -> unconnected-(Y2-NC-Pad3)
- Y2 pad 4: /+3V3_DIG -> GND
Routing:
- net /RX_MCU_CLOCK/TCXO_10M: track 21.4 -> 0.00 mm
- net /RX_MCU_CLOCK/REF_10M: track 0.00 -> 16.3 mm, vias 0 -> 2
- net /+3V3_DIG: track 282.4 -> 269.3 mm, vias 0 -> 3
- net /HOST_I2C_SDA: track 35.0 -> 43.3 mm, vias 0 -> 2
- net /PPS_OUT: track 60.2 -> 66.8 mm, vias 0 -> 2
- net /HOST_I2C_SCL: track 37.3 -> 43.9 mm
- net GND: track 100.4 -> 104.9 mm, vias 50 -> 52
- net Net-(U4-XOUT): track 13.0 -> 13.7 mm
- net Net-(U4-XIN): track 22.8 -> 23.5 mm
- net /HOST_READY: track 58.0 -> 58.6 mm

Commit message: manufacturing files
Parts:
- J2: footprint Connector_JST:JST_PH_B8B-PH-K_1x08_P2.00mm_Vertical -> Connector_PinHeader_2.54mm:PinHeader_1x08_P2.54mm_Vertical
- moved D1 3.20 mm to (131.6, 106.7)
- moved J2 1.61 mm to (130.5, 87.9), turned to 0 degrees
Routing:
- net /HOST_READY: track 58.6 -> 65.9 mm
- net /+3V3_DIG: track 269.3 -> 275.9 mm
- net GND: track 104.9 -> 108.9 mm
- net /RX_OPTICAL_AFE/PD_SUM_NODE: track 5.60 -> 8.93 mm
- net /HOST_I2C_SCL: track 43.9 -> 46.5 mm
- net /PPS_OUT: track 66.8 -> 64.8 mm
- net /HOST_UART_RX: track 32.7 -> 34.7 mm
- net /RX_POWER_USB/VIN_HOST_5V: track 12.6 -> 10.9 mm
- net /HOST_UART_TX: track 32.1 -> 33.8 mm
- net /HOST_I2C_SDA: track 43.3 -> 44.5 mm
