File: fsoc-rx/rx_power_usb.kicad_sch (KiCad schematic)
At the start: 12 parts, among them J1 USB4105-GF-A, J2 B8B-PH-K-S, U1 USBLC6-2SC6, U2 AP2112K-3.3, U3 TPS7A2033PDBVR

Commit message: RX ROOT: optical AFE
Parts:
- renumbered C3 to C1, C1 to C2, C4 to C3, C2 to C4
Changed lines of the file:
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@@
+	)
+	(junction
+		(at 210.82 97.79)
+		(diameter 0)
+		(color 0 0 0 0)
 	)
 	(junction
@@
 		(color 0 0 0 0)
 	)
-	(junction
-		(at 210.82 97.79)
-		(diameter 0)
-		(color 0 0 0 0)
-	)
 	(no_connect
 		(at 99.06 107.95)
@@
 	(wire
 		(pts
-			(xy 153.67 85.09) (xy 152.4 85.09)
+			(xy 156.21 85.09) (xy 152.4 85.09)
 		)
 		(stroke
@@
 	(label "VBUS_USB"
 		(at 134.62 72.39 0)
+		(effects
+			(font
+				(size 1.27 1.27)
+			)
+			(justify left bottom)
+		)
+	)
+	(label "SYS_5V"
+		(at 156.21 85.09 0)
 		(effects
 			(font
@@
 			)
 			(justify right)
-		)
-	)
-	(hierarchical_label "SYS_5V"
-		(shape output)
-		(at 153.67 85.09 0)
-		(effects
-			(font
-				(size 1.27 1.27)
-			)
-			(justify left)
 		)
 	)
@@
 		(dnp no)
 		(fields_autoplaced yes)
-		(property "Reference" "#PWR011"
+		(property "Reference" "#PWR010"
 			(at 236.22 83.82 0)
 			(hide yes)
@@
 			(project "fsoc-rx"
 				(path "/84f983f4-ce6f-4382-bffe-129758307136/e570b0c0-cac5-4a7f-a320-8fd087761133"
-					(reference "#PWR011")
+					(reference "#PWR010")
 					(unit 1)
 				)
@@
 		(dnp no)
 		(fields_autoplaced yes)
-		(property "Reference" "#PWR05"
+		(property "Reference" "#PWR07"
 			(at 210.82 111.76 0)
 			(hide yes)
@@
 			(project "fsoc-rx"
 				(path "/84f983f4-ce6f-4382-bffe-129758307136/e570b0c0-cac5-4a7f-a320-8fd087761133"
-					(reference "#PWR05")
+					(reference "#PWR07")
 					(unit 1)
 				)
@@
 		(dnp no)
 		(fields_autoplaced yes)
-		(property "Reference" "#PWR03"
+		(property "Reference" "#PWR04"
 			(at 121.92 107.95 0)
 			(hide yes)
@@
 			(project "fsoc-rx"
 				(path "/84f983f4-ce6f-4382-bffe-129758307136/e570b0c0-cac5-4a7f-a320-8fd087761133"
-					(reference "#PWR03")
+					(reference "#PWR04")
 					(unit 1)
 				)
@@
 		(dnp no)
 		(fields_autoplaced yes)
-		(property "Reference" "#PWR08"
+		(property "Reference" "#PWR01"
 			(at 76.2 121.92 0)
 			(hide yes)
@@
 			(project "fsoc-rx"
 				(path "/84f983f4-ce6f-4382-bffe-129758307136/e570b0c0-cac5-4a7f-a320-8fd087761133"
-					(reference "#PWR08")
+					(reference "#PWR01")
 					(unit 1)
 				)
@@
 		(dnp no)
 		(fields_autoplaced yes)
-		(property "Reference" "#PWR04"
+		(property "Reference" "#PWR05"
 			(at 148.59 109.22 0)
 			(hide yes)
@@
 			(project "fsoc-rx"
 				(path "/84f983f4-ce6f-4382-bffe-129758307136/e570b0c0-cac5-4a7f-a320-8fd087761133"
-					(reference "#PWR04")
+					(reference "#PWR05")
 					(unit 1)
 				)
@@
 		(dnp no)
 		(fields_autoplaced yes)
-		(property "Reference" "#PWR06"
+		(property "Reference" "#PWR011"
 			(at 236.22 111.76 0)
 			(hide yes)
@@
 			(project "fsoc-rx"
 				(path "/84f983f4-ce6f-4382-bffe-129758307136/e570b0c0-cac5-4a7f-a320-8fd087761133"
-					(reference "#PWR06")
+					(reference "#PWR011")
 					(unit 1)
 				)
@@
 		(dnp no)
 		(fields_autoplaced yes)
-		(property "Reference" "C2"
+		(property "Reference" "C4"
 			(at 240.03 100.3299 0)
 			(show_name no)
@@
 			(project "fsoc-rx"
 				(path "/84f983f4-ce6f-4382-bffe-129758307136/e570b0c0-cac5-4a7f-a320-8fd087761133"
-					(reference "C2")
+					(reference "C4")
 					(unit 1)
 				)
@@
 		(dnp no)
 		(fields_autoplaced yes)
-		(property "Reference" "#PWR010"
+		(property "Reference" "#PWR06"
 			(at 208.28 83.82 0)
 			(hide yes)
@@
 			(project "fsoc-rx"
 				(path "/84f983f4-ce6f-4382-bffe-129758307136/e570b0c0-cac5-4a7f-a320-8fd087761133"
-					(reference "#PWR010")
+					(reference "#PWR06")
 					(unit 1)
 				)
@@
 		(in_pos_files yes)
 		(dnp no)
-		(property "Reference" "C1"
+		(property "Reference" "C2"
 			(at 205.232 99.822 0)
 			(show_name no)
@@
 			(project "fsoc-rx"
 				(path "/84f983f4-ce6f-4382-bffe-129758307136/e570b0c0-cac5-4a7f-a320-8fd087761133"
-					(reference "C1")
+					(reference "C2")
 					(unit 1)
 				)
@@
 		(dnp no)
 		(fields_autoplaced yes)
-		(property "Reference" "C4"
+		(property "Reference" "C3"
 			(at 240.03 72.3899 0)
 			(show_name no)
@@
 			(project "fsoc-rx"
 				(path "/84f983f4-ce6f-4382-bffe-129758307136/e570b0c0-cac5-4a7f-a320-8fd087761133"
-					(reference "C4")
+					(reference "C3")
 					(unit 1)
 				)
@@
 		(dnp no)
 		(fields_autoplaced yes)
-		(property "Reference" "C3"
+		(property "Reference" "C1"
 			(at 212.09 71.1199 0)
 			(show_name no)
@@
 			(project "fsoc-rx"
 				(path "/84f983f4-ce6f-4382-bffe-129758307136/e570b0c0-cac5-4a7f-a320-8fd087761133"
-					(reference "C3")
+					(reference "C1")
 					(unit 1)
 				)
@@
 		(dnp no)
 		(fields_autoplaced yes)
-		(property "Reference" "#PWR01"
+		(property "Reference" "#PWR03"
 			(at 113.03 90.17 0)
 			(hide yes)
@@
 			(project "fsoc-rx"
 				(path "/84f983f4-ce6f-4382-bffe-129758307136/e570b0c0-cac5-4a7f-a320-8fd087761133"
-					(reference "#PWR01")
+					(reference "#PWR03")
 					(unit 1)
 				)
@@
 		(dnp no)
 		(fields_autoplaced yes)
-		(property "Reference" "#PWR07"
+		(property "Reference" "#PWR08"
 			(at 223.52 111.76 0)
 			(hide yes)
@@
 			(project "fsoc-rx"
 				(path "/84f983f4-ce6f-4382-bffe-129758307136/e570b0c0-cac5-4a7f-a320-8fd087761133"
-					(reference "#PWR07")
+					(reference "#PWR08")
 					(unit 1)
 				)

Commit message: RX: footprint assignments
Parts:
- C1, C2, C3, C4: footprint (none) -> Capacitor_SMD:C_0805_2012Metric
- R1, R2: footprint (none) -> Resistor_SMD:R_0603_1608Metric
Changed lines of the file:
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@@
 			)
 		)
-		(property "Footprint" ""
+		(property "Footprint" "Resistor_SMD:R_0603_1608Metric"
 			(at 102.87 84.328 90)
 			(hide yes)
@@
 			)
 		)
-		(property "Footprint" ""
+		(property "Footprint" "Resistor_SMD:R_0603_1608Metric"
 			(at 102.87 86.868 90)
 			(hide yes)
@@
 			)
 		)
-		(property "Footprint" ""
+		(property "Footprint" "Capacitor_SMD:C_0805_2012Metric"
 			(at 237.1852 105.41 0)
 			(hide yes)
@@
 			)
 		)
-		(property "Footprint" ""
+		(property "Footprint" "Capacitor_SMD:C_0805_2012Metric"
 			(at 211.7852 105.41 0)
 			(hide yes)
@@
 			)
 		)
-		(property "Footprint" ""
+		(property "Footprint" "Capacitor_SMD:C_0805_2012Metric"
 			(at 237.1852 77.47 0)
 			(hide yes)
@@
 			)
 		)
-		(property "Footprint" ""
+		(property "Footprint" "Capacitor_SMD:C_0805_2012Metric"
 			(at 209.2452 76.2 0)
 			(hide yes)

Commit message: RX PCB
Parts:
- J1: footprint Connector_USB:USB_C_Receptacle_GCT_USB4105-xx-A_16P_TopMnt_Horizontal -> fsoc_footprints:TYPE-C-31-M-14
Connections:
- net USB_CONN_DP: now reaches J1.A6 (D+), J1.B6 (D+), U1.3 (I/O2)
- net USB_CONN_DN: now reaches J1.A7 (D-), J1.B7 (D-), U1.1 (I/O1)
- net USB_DM renamed USB_DN
Changed lines of the file:
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@@
+		)
+	)
+	(label "USB_CONN_DP"
+		(at 102.87 97.79 0)
+		(effects
+			(font
+				(size 1.27 1.27)
+			)
+			(justify left bottom)
 		)
 	)
 	(label "VBUS_USB"
 		(at 109.22 72.39 0)
+		(effects
+			(font
+				(size 1.27 1.27)
+			)
+			(justify left bottom)
+		)
+	)
+	(label "USB_CONN_DN"
+		(at 102.87 92.71 0)
 		(effects
 			(font
@@
 		)
 	)
-	(hierarchical_label "USB_DM"
+	(hierarchical_label "USB_DN"
 		(shape bidirectional)
 		(at 134.62 90.17 0)
@@
 			)
 		)
-		(property "Footprint" "Connector_USB:USB_C_Receptacle_GCT_USB4105-xx-A_16P_TopMnt_Horizontal"
+		(property "Footprint" "fsoc_footprints:TYPE-C-31-M-14"
 			(at 87.63 92.71 0)
 			(hide yes)

Commit message: manufacturing files
Parts:
- J2: footprint Connector_JST:JST_PH_B8B-PH-K_1x08_P2.00mm_Vertical -> Connector_PinHeader_2.54mm:PinHeader_1x08_P2.54mm_Vertical
Changed lines of the file:
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@@
 			)
 		)
-		(property "Footprint" "Connector_JST:JST_PH_B8B-PH-K_1x08_P2.00mm_Vertical"
+		(property "Footprint" "Connector_PinHeader_2.54mm:PinHeader_1x08_P2.54mm_Vertical"
 			(at 176.53 106.68 0)
 			(hide yes)
